File: pcb/ps2_serial.kicad_pcb (KiCad board)
At the start: 2 copper layers, 97 x 76 mm, 37 parts, among them J1 Jumper 1, J2 Conn_01x06, J3 serial header, J4 SPI, J5 USB_A, J6 power, Q1 Q_PMOS_GDS, U1 ATtiny2313-20P, U2 MAX232, Y1 Crystal_Small

Commit message: V2 for PCB. Implemented following changes: -more elegant mounting mechanism -more jumper settings -footprint for both USB and PS/2 socket -reservation for using INT0 to trigger SDA sampling -smaller size board
Parts:
- removed H1, H2: MountingHole_Pad, MountingHole:MountingHole_4.3mm_M4_DIN965_Pad
- removed J2: Conn_01x06, Connector_PinHeader_2.54mm:PinHeader_1x06_P2.54mm_Vertical
- added C10: 33p, Capacitor_THT:C_Disc_D4.3mm_W1.9mm_P5.00mm, F.Cu at (189.0, 102.0)
- added J10: Mini-DIN-6, kicad:J_Mini-DIN-6, F.Cu at (219.0, 55.0)
- added J11: Conn_01x03, Connector_PinHeader_2.54mm:PinHeader_1x03_P2.54mm_Vertical, F.Cu at (233.9, 75.0)
- added J12: Screw_Terminal_01x01, Amphenol:Amphenol_M4-44051DB, F.Cu at (191.8, 62.5)
- added J13: Screw_Terminal_01x01, Amphenol:Amphenol_M4-44051DB, F.Cu at (254.8, 62.5)
- added R13: 0, Resistor_THT:R_Axial_DIN0207_L6.3mm_D2.5mm_P10.16mm_Horizontal, F.Cu at (192.0, 82.1)
- C6: value 220u -> 330u; footprint Capacitor_THT:CP_Radial_D10.0mm_P5.00mm -> Capacitor_THT:CP_Radial_D8.0mm_P3.50mm
- C8, C9: value 22p -> 33p
- D2, D3, D4: value ZPYxx -> P6KE6.8
- J1: value Jumper 1 -> Jumper; footprint Connector_PinHeader_2.54mm:PinHeader_1x03_P2.54mm_Vertical -> Connector_PinHeader_2.54mm:PinHeader_2x05_P2.54mm_Vertical
- Q1: footprint Package_TO_SOT_SMD:TO-263-2 -> Package_TO_SOT_SMD:TO-252-2
- R9: value 47k -> 39k
- Y1: value Crystal_Small -> 18.432M
- moved D2 16.1 mm to (229.9, 84.0)
- moved Q1 13.4 mm to (204.5, 65.9), turned to 90 degrees
- moved R7 12.9 mm to (214.3, 73.0)
- moved R12 11.3 mm to (216.9, 78.0), turned to 0 degrees
- moved R2 10.3 mm to (233.0, 104.1)
- moved R3 10.3 mm to (238.0, 104.1)
- moved J9 9.00 mm to (241.5, 68.4)
- moved D4 8.51 mm to (246.9, 75.0), turned to 0 degrees
- moved D1 5.29 mm to (195.0, 74.2)
- moved D3 5.00 mm to (240.1, 79.0)
- moved J1 3.62 mm to (182.5, 101.8)
- moved R11 3.54 mm to (209.5, 85.4)
- moved C8 3.00 mm to (186.5, 96.5)
- moved C9 3.00 mm to (186.5, 91.5)
- moved Y1 3.00 mm to (191.0, 91.6)
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- renumbered J3 to J7, J4 to J8, J5 to J9
Connections:
- J1 pad 1: Net-(J1-Pin_1) -> GND
- J1 pad 3: Net-(J1-Pin_3) -> GND
- U1 pad 11: unconnected-(U1-PD6-Pad11) -> Net-(J1-Pin_10)
- U1 pad 2: VCC -> Net-(J1-Pin_2)
- U1 pad 6: unconnected-(U1-PD2-Pad6) -> Net-(U1-PD2)
- U1 pad 7: Net-(J1-Pin_1) -> Net-(J1-Pin_4)
- U1 pad 8: Net-(J1-Pin_2) -> Net-(J1-Pin_6)
- U1 pad 9: Net-(J1-Pin_3) -> Net-(J1-Pin_8)
Routing:
- net Net-(U1-PD2): track 0.00 -> 50.3 mm, vias 0 -> 1
- net /PS/2 data: track 28.2 -> 59.8 mm
- net VCC: track 207.3 -> 176.7 mm, vias 1 -> 0
- net Net-(J1-Pin_10): track 0.00 -> 21.3 mm, vias 0 -> 1
- net /PS/2 clock: track 36.7 -> 53.0 mm
- net Net-(J1-Pin_3): track 15.8 -> 0.00 mm
- net Net-(J1-Pin_1): track 15.8 -> 0.00 mm
- net Net-(J1-Pin_2): track 15.8 -> 30.3 mm
- net Net-(Q1-S): track 101.4 -> 87.7 mm
- net Net-(J1-Pin_6): track 0.00 -> 12.8 mm
- net Net-(J1-Pin_4): track 0.00 -> 12.8 mm
- net Net-(J1-Pin_8): track 0.00 -> 12.8 mm
- net Net-(U1-PB1): track 46.2 -> 35.0 mm
- net /SDA/MOSI: track 83.9 -> 74.6 mm
- net /SCL: track 73.2 -> 65.4 mm
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- added copper zone on F.Cu, net GND
- added copper zone on B.Cu, net Net-(Q1-D)
Other:
- board size 97 x 76 mm -> 97 x 67 mm
- board text added: "J2"
- board text added: "J3"
- board text added: "J4"
- board text added: "J5"
- board text added: "PS/2 to serial converter V2"
